File: project.kicad_sch (KiCad schematic)
At the start: 3 parts, among them U1 WLC1115-68LQXQ

Commit message: started schem
Parts:
- added C3, C4: C, symbol Device:C
- added C5, C7: 0.1u, symbol Device:C
- added C6, C8: 1u, symbol Device:C
- added D1, D2: LED, symbol Device:LED
- added J1: Conn_01x05_Pin, symbol Connector:Conn_01x05_Pin
- added J2, J3: Conn_01x01_Pin, symbol Connector:Conn_01x01_Pin
- added R1: R, symbol Device:R
- added R2, R3: 4.7k, symbol Device:R
- added R4, R6, R7: 1k, symbol Device:R
- added R5: 2k, symbol Device:R
- added U2: SLS32AIA020U2USON10XTMA1, PG-USON-10-2, symbol Optiga Trust:SLS32AIA020U2USON10XTMA1
Connections:
- net GND: now also U1.34 (GND), U1.64 (GND), U1.69 (EPAD), C3.1, C4.1, C5.1, C6.1, C7.1, C8.1, J1.5 (Pin_5), R5.2, R6.1, R7.1, U2.1 (GND)
- net VBUS: now also U1.39 (VBUS_IN)
- net at U1.10 (COMP): now also C3.2, R1.2
- net at U1.20 (PWM_IN1): now also U1.21 (PWM_IN2), U1.22 (PWM_OUT)
- net +5V: now reaches U1.25 (VDDD)
- net +5V: now also U1.63 (VDDD), C5.2, C6.2, C7.2, C8.2, J1.1 (Pin_1), R2.1, R3.2, U2.10 (VCC)
- net at U1.27 (LED2): now also D2.2 (A)
- net reset: now reaches U1.28 (*XRES)
- net reset: now also J1.4 (Pin_4)
- net at U1.29 (SDA_SEC): now also U2.3 (SDA)
- net at U1.30 (SCL_SEC): now also U2.8 (SCL)
- net at U1.31 (UART/GPIO7): now also J2.1 (Pin_1)
- net at U1.33 (RES_SEC): now also U2.9 (RST)
- net VBB: now reaches U1.38 (BB_IN)
- net at U1.56 (SWD_DAT/GPIO9): now also J1.3 (Pin_3), R2.2
- net at U1.57 (SWD_CLK/GPIO10): now also J1.2 (Pin_2), R3.1
- net at U1.58 (TEMP_FB): now also J3.1 (Pin_1)
- net at U1.59 (GPIO12): now also R4.1
- new net: D2.1 (K), R7.2
- new net: C4.2, R1.1
- new net: D1.1 (K), R6.2
- new net COMM: R4.2, R5.1
Other:
- moved on the sheet: C1, C2

Commit message: added reference doc
Parts:
- added C10, C11, C12, C13, C14, C15, C16, C9: C, symbol Device:C
- added D3, D4, D5, D6, D7: D, symbol Device:D
- added Q1: BSZ0902NS, NFET:IFX-PG-TSDSON-8-26-V, symbol NFET:BSZ0902NS
- added R10, R11, R12, R13, R14, R15, R16, R17, R18, R19, R8, R9: R, symbol Device:R
Connections:
- net +5V: now also R13.1
- net GND: now also C10.2, C12.2, C14.1, D3.1 (K), D4.2 (A), R10.2, R12.2, R17.1
- net VBB: now also Q1.1 (SOURCE), Q1.2 (SOURCE), Q1.3 (SOURCE)
- net VBUS: now also Q1.5 (DRAIN), Q1.6 (DRAIN), Q1.7 (DRAIN), Q1.8 (DRAIN)
- net at U1.26 (LED1): now also D1.2 (A)
- net optigaSDA: now reaches U1.29 (SDA_SEC), U2.3 (SDA)
- net optigaSCL: now reaches U1.30 (SCL_SEC), U2.8 (SCL)
- net QComp: now reaches U1.32 (QCOMP2)
- net QComp: now also U1.37 (QCOMP1), R10.1, R9.2
- net optigaRST: now reaches U1.33 (RES_SEC), U2.9 (RST)
- net NFet Control: now reaches U1.35 (NFET_CTRL_1)
- net NFet Control: now also Q1.4 (GATE)
- net ASK_N: now reaches U1.40 (ASK_N)
- net ASK_N: now also C12.1, C13.2, R16.2
- net ASK_P: now reaches U1.41 (ASK_P)
- net ASK_P: now also C13.1, C14.2, R15.2
- new net: R13.2, R14.1, R15.1
- new net: D6.1 (K), D7.2 (A)
- new net: C16.2, D6.2 (A), D7.1 (K), R19.1
- new net: C10.1, C11.1, D5.1 (K), R12.1
- new net: C15.1, C16.1, R18.2
- new net: D5.2 (A), R11.2
- new net: D3.2 (A), D4.1 (K), R8.2, R9.1
- new net: C9.2, R8.1
- new net: C11.2, R14.2, R16.1, R17.2
- new net COIL_SNS: C9.1, R11.1
Other:
- note added: "Optiga Security Chip"
- note added: "Power NFet"
- note added: "Q Estimate Circuit"
- moved on the sheet: U2

Commit message: fr
Parts:
- removed D5, D6, D7: D, symbol Device:D
- added C17, C19: 0.1u, symbol Device:C
- added C18: 1u, symbol Device:C
- added C20, C21, C22: C, symbol Device:C
- added D5, D6: Diode, symbol bat54s:Diode-NC_pin
- added D7: BAT64T5Q-7-F, SODFL1608X65N, symbol bat64t:BAT64T5Q-7-F
- added D8, D9: RB511SM-40FHT2R, RB511SM40FHT2R, symbol rb511sm:RB511SM-40FHT2R
- added J4: Conn_01x05_Socket, symbol Connector:Conn_01x05_Socket
- added L1: PA4342.682NLT, ProtoFlow.pretty:Yageo_Pulse_PA4342_10.3x11.5mm, symbol PA4342.682NLT:PA4342.682NLT
- added Q2, Q3: BSZ0902NS, symbol NFET:BSZ0902NS
- added R20, R21: 5.1k, symbol Device:R
- added R22: R, symbol Device:R
- added TP1: TestPoint_Probe, symbol Connector:TestPoint_Probe
- added TP2: OPAMP_GAIN, symbol Connector:TestPoint_Probe
- added TP3: OPAMP_CMP, symbol Connector:TestPoint_Probe
- added TP4: CMP_REF, symbol Connector:TestPoint_Probe
- added TP5: PVIN_0, symbol Connector:TestPoint_Probe
- added TP6: HG1_0, symbol Connector:TestPoint_Probe
- added TP7: LG1_0, symbol Connector:TestPoint_Probe
- added TP8: SW1_0, symbol Connector:TestPoint_Probe
- added U3: LMV358AQDGKRQ1, DGK8_TEX, symbol opamp:LMV358AQDGKRQ1
- C10: value C -> 22nf
- C11: value C -> 0.22uf
- C12: value C -> 22n
- C13: value C -> 0.1u
- C14: value C -> 330p; now not fitted
- C15: value C -> 150p
- C16: value C -> 10n; now not fitted
- R11: value R -> 1k
- R12: value R -> 27k
- R13: value R -> 5.1k
- R14: value R -> 390
- R15: value R -> 10k
- R16: value R -> 100k
- R17: value R -> 0
- R18: value R -> 1M; now not fitted
- R19: value R -> 10k; now not fitted
Connections:
- net optigaRST is gone; now on net OPTIGA_I2C_INT: U1.33 (RES_SEC), U2.9 (RST)
- net +5V: no longer R13.1, U2.10 (VCC)
- net ASK_N: no longer C12.1, C13.2, R16.2
- net ASK_P: no longer C13.1, C14.2, R15.2
- net COIL_SNS: no longer R11.1
- net GND: now also C13.2, C16.1, R15.2, C17.2, C18.1, C19.2, C20.2, C21.2, J4.4 (Pin_4), Q3.1 (SOURCE), Q3.2 (SOURCE), Q3.3 (SOURCE), U3.4 (V-); no longer R12.2, R17.1
- net at C16.2: now also R17.2, R18.1, U3.5 (+INB); no longer R19.1
- net at C10.1, C11.1: now also R11.2; no longer R12.1
- net ASK_OUT: now reaches U1.18 (ASK_OUT)
- net ASK_OUT: now also R11.1, TP1.1
- net ASK_DEMOD: now reaches U1.19 (ASK_DEMOD)
- net ASK_DEMOD: now also R18.2, TP3.1, U3.7 (OUTB)
- net at C15.2: now also R16.2, R17.1, TP2.1, U3.1 (OUTA)
- net OPTIGA_I2C_INT: now reaches R19.2
- net optigaSCL renamed OPTIGA_I2C_SCL
- net OPTIGA_I2C_SCL: now also R20.2
- net optigaSDA renamed OPTIGA_I2C_SDA
- net OPTIGA_I2C_SDA: now also R21.2
- new net: C14.2, C15.1, R13.2, R16.1, U3.2 (-INA)
- new net: C12.1, D5.2 (C), D6.1 (A), R12.2, R14.1, U3.3 (+INA)
- new net: C13.1, R14.2, R15.1, TP4.1, U3.6 (-INB)
- new net: C19.1, D7.2 (A), J4.5 (Pin_5)
- new net: C11.2, D5.1 (A), D6.2 (C), R13.1
- new net BST1_0: C22.2, D8.1 (K)
- new net BST2_0: D9.1 (K)
- new net HG1_0: Q2.4 (GATE), TP6.1
- new net HPI_I2C_SCL: J4.2 (Pin_2)
- new net HPI_I2C_SDA: J4.1 (Pin_1)
- new net IIN_CSN_0: Q2.5 (DRAIN), Q2.6 (DRAIN), Q2.7 (DRAIN), Q2.8 (DRAIN), R22.2
- new net LG1_0: Q3.4 (GATE), TP7.1
- new net PVIN_0: C20.1, C21.1, R22.1, TP5.1
- new net SW1_0: C22.1, L1.1, Q2.1 (SOURCE), Q2.2 (SOURCE), Q2.3 (SOURCE), Q3.5 (DRAIN), Q3.6 (DRAIN), Q3.7 (DRAIN), Q3.8 (DRAIN), TP8.1
- new net VDDD: C17.1, C18.2, D7.1 (K), D8.2 (A), D9.2 (A), R12.1, R19.1, R20.1, R21.1, U2.10 (VCC), U3.8 (V+)
- new net XRES: J4.3 (Pin_3)
Other:
- note added: "ASK Demodulation"
- moved on the sheet: C1, C2, C3, C4, C5, C6, C7, C8, D1, D2, J1, J2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

Commit message: fixing remote
Parts:
- removed J1: Conn_01x05_Pin, symbol Connector:Conn_01x05_Pin
- added C23, C24, C25, C26, C29, C30: 22u, symbol Device:C
- added C27: 4.7u, symbol Device:C
- added C28, C33, C41: 10n, symbol Device:C
- added C31, C32, C34, C35, C36, C37, C38, C39, C40: 0.1u, symbol Device:C
- added D10, D11: RB511SM-40FHT2R, RB511SM40FHT2R, symbol rb511sm:RB511SM-40FHT2R
- added L2: MP-A11, symbol Device:L
- added Q4, Q5, Q6, Q7: BSZ0902NS, symbol NFET:BSZ0902NS
- added R23: 0.01, symbol Device:R
- added R24: 0, symbol Device:R
- added TP10: LG2_1, symbol Connector:TestPoint_Probe
- added TP11: COIL_SNS, symbol Connector:TestPoint_Probe
- added TP12: HG1_1, symbol Connector:TestPoint_Probe
- added TP13: LG1_1, symbol Connector:TestPoint_Probe
- added TP14: SW2_1, symbol Connector:TestPoint_Probe
- added TP15: SW1_1, symbol Connector:TestPoint_Probe
- added TP9: HG2_1, symbol Connector:TestPoint_Probe
- C20, C21: value C -> 22u
- C22: value C -> 0.1u
- R2: value 4.7k -> 5.1k
- R22: value R -> 0.005
- R3: value 4.7k -> 0
Connections:
- net COIL_SNS: now also C34.2, C35.2, C36.2, C37.2, C38.2, L2.1, TP11.1
- net GND: now also R3.2, C23.2, C24.2, C25.2, C26.2, C27.2, C28.2, C29.2, C30.2, C31.2, C32.2, Q5.1 (SOURCE), Q5.2 (SOURCE), Q5.3 (SOURCE), Q7.1 (SOURCE), Q7.2 (SOURCE), Q7.3 (SOURCE), R24.2
- net IIN_CSN_0: now also C27.1, C28.1
- net VDDD: now also C5.2, C6.2, C7.2, C8.2, R2.2, U1.25 (VDDD), U1.63 (VDDD), D10.2 (A), D11.2 (A)
- net at U1.56 (SWD_DAT/GPIO9): no longer R2.2
- net at U1.57 (SWD_CLK/GPIO10): no longer R3.1
- net IOUT_CSP_0: now reaches L1.2
- net IOUT_CSP_0: now also C23.1, C24.1, C25.1, C26.1, R23.1
- removed net +5V: C5.2, C6.2, C7.2, C8.2, R2.1, R3.2, U1.25 (VDDD), U1.63 (VDDD)
- new net: C41.2, R24.1
- new net: C33.2, R3.1
- new net BST1_1: C40.1, D11.1 (K)
- new net BST2_1: C39.1, D10.1 (K)
- new net HG1_1: Q6.4 (GATE), TP12.1
- new net HG2_1: Q4.4 (GATE), TP9.1
- new net LG1_1: Q7.4 (GATE), TP13.1
- new net LG2_1: Q5.4 (GATE), TP10.1
- new net SW1_1: C40.2, C41.1, L2.2, Q6.1 (SOURCE), Q6.2 (SOURCE), Q6.3 (SOURCE), Q7.5 (DRAIN), Q7.6 (DRAIN), Q7.7 (DRAIN), Q7.8 (DRAIN), TP15.1
- new net SW2_1: C33.1, C34.1, C35.1, C36.1, C37.1, C38.1, C39.2, Q4.1 (SOURCE), Q4.2 (SOURCE), Q4.3 (SOURCE), Q5.5 (DRAIN), Q5.6 (DRAIN), Q5.7 (DRAIN), Q5.8 (DRAIN), TP14.1
- new net VBB_1: C29.1, C30.1, C31.1, C32.1, Q4.5 (DRAIN), Q4.6 (DRAIN), Q4.7 (DRAIN), Q4.8 (DRAIN), Q6.5 (DRAIN), Q6.6 (DRAIN), Q6.7 (DRAIN), Q6.8 (DRAIN), R23.2
Other:
- note added: "Buck Convertor"
- note added: "Full Bridge Inverter"
- moved on the sheet: C19, C20, C21, C22, C9, D3, D4, D7, D8, D9, J4, L1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

Commit message: fixed some things
Parts:
- added C42, C44: 1u, symbol Device:C
- added C43, C45: 0.1u, symbol Device:C
- added R25, R26, R29, R30: 0, symbol Device:R
- added R27, R28: 10, symbol Device:R
- added R31: 5.1k, symbol Device:R
- added TP16: Vin, symbol Connector:TestPoint_Probe
- added TP17: VDDD, symbol Connector:TestPoint_Probe
- added TP18: VBRG_0, symbol Connector:TestPoint_Probe
- C2: value 1u -> 2.2u
- C3: value C -> 1n
- C4: value C -> 0.47n
- C8: value 1u -> 0.1u
- R1: value R -> 1k
Connections:
- net reset is gone; now on net XRES: U1.28 (*XRES)
- net ASK_DEMOD: now also U1.36 (ASK_SEL)
- net BST1_0: now also U1.67 (BST1_0)
- net GND: now also C42.1, C43.1, C44.1, C45.1; no longer C2.2
- net HG1_0: now also U1.68 (HG1_0)
- net HPI_I2C_SCL: now also U1.57 (SWD_CLK/GPIO10), R31.1
- net HPI_I2C_SDA: now also R2.1, U1.56 (SWD_DAT/GPIO9)
- net IIN_CSN_0: now also U1.66 (CSNI_0)
- net PVIN_0: now also U1.65 (CSPI_0), R25.1
- net VBB_1: now also R28.1
- net VBUS: no longer U1.61 (VIN)
- net VDDD: now also R26.1, R31.2; no longer C7.2, C8.2, U1.63 (VDDD)
- net at U1.11 (CSPO): now also C2.1, R27.2
- net at U1.12 (CSNO): now also C2.2, R28.2
- net at U1.13 (VBRG): now also C7.2, R29.2
- net at U1.14 (VBRG_DIS): now also C8.2, R30.2
- net toESP: now reaches R4.1, U1.59 (GPIO12)
- net at C1.1, U1.62 (VCCD): no longer C2.1
- net IOUT_CSP_0 renamed VBRG_0
- net VBRG_0: now also R27.1, R29.1, R30.1, TP18.1
- new net VDDD_in: C44.2, C45.2, R26.2, TP17.1, U1.63 (VDDD)
- new net Vin: C42.2, C43.2, R25.2, TP16.1, U1.61 (VIN)
Other:
- note added: "IC -> ESP"
- note added: "Power In"
- note added: "Programming Connector"
- moved on the sheet: C1, C3, C4, R1

Commit message: added provided gerber
Parts:
- removed C9: C, symbol Device:C
- removed D3, D4: D, symbol Device:D
- removed J2: Conn_01x01_Pin, symbol Connector:Conn_01x01_Pin
- removed R10: R, symbol Device:R
- added C46, C48: 10n, symbol Device:C
- added C47: 470n, symbol Device:C
- added C49, C53, C54: 0.1u, symbol Device:C
- added C50: 100n, symbol Device:C
- added C51: 5.6n, symbol Device:C
- added C52: 1n, symbol Device:C
- added D12: 1N4448W-TP, SOD3716X135N, symbol 1N4448W-TP:1N4448W-TP
- added D13: MMBD1503A, SOT95P240X120-3N, symbol MMBD1503A:MMBD1503A
- added J1: Conn_01x02_Pin, symbol Connector:Conn_01x02_Pin
- added Q8: BSS138N, Package_TO_SOT_SMD:SOT-23, symbol Transistor_FET:BSS138
- added R32, R33: 10, symbol Device:R
- added R34: 62, symbol Device:R
- added R35: 2.2k, symbol Device:R
- added R36: 130k, symbol Device:R
- added R37, R43: 0, symbol Device:R
- added R38: 100k, symbol Device:R
- added R39: 5.1k, symbol Device:R
- added R40: 36k, symbol Device:R
- added R41: 3.6k, symbol Device:R
- added R42: 20k, symbol Device:R
- added TP19: V2I_IP, symbol Connector:TestPoint_Probe
- added TP20: Q_COMP, symbol Connector:TestPoint_Probe
- added TP21: PWN_OUT, symbol Connector:TestPoint_Probe
- R8, R9: value R -> 0
Connections:
- net VBRG_0 is gone; now on net IOUT_CSP_0: C23.1, C24.1, C25.1, C26.1, L1.2, R23.1, R27.1, R29.1, R30.1, TP18.1
- net ASK_N: now also C47.1, C48.1, R33.1
- net ASK_P: now also C46.1, C47.2, R32.1
- net BST2_0: now also U1.9 (BST2_0)
- net COIL_SNS: now also C52.2, R39.2
- net GND: now also R8.1, C46.2, C48.2, C49.1, C51.1, C53.2, C54.2, D13.2 (CATHODE), J1.2 (Pin_2), R36.1, R38.1, R42.2
- net PVIN_0: now also U1.38 (BB_IN), U1.39 (VBUS_IN), C53.1, C54.1
- net QComp: no longer R9.2
- net VBB: no longer U1.38 (BB_IN)
- net VBUS: no longer U1.39 (VBUS_IN)
- net VDDD: now also D13.1 (ANODE), Q8.1 (G), R35.2
- net at U1.20 (PWM_IN1), U1.21 (PWM_IN2), U1.22 (PWM_OUT): now also TP21.1
- net at U1.31 (UART/GPIO7): now also J1.1 (Pin_1)
- net at U1.6 (VBB_0): now also R9.2
- net at U1.7 (SW2_0): now also R8.2
- net IOUT_CSP_0: now reaches R9.1
- net IOUT_CSP_0: no longer R8.2
- new net: D12.2 (A), R39.1
- new net: C52.1, R40.1
- new net: Q8.3 (D), R41.2, R42.1, R43.1
- new net: C50.1, R37.1
- new net: D13.3 (A_/_C), R40.2, R41.1
- new net ASK_I_N: C49.2, C50.2, R33.2, R34.1, R36.2, TP19.1
- new net ASK_I_P: R32.2, R34.2, R35.1
- new net ASK_PEAK: C51.2, D12.1 (K), R37.2, R38.2
- new net Q_COMP: Q8.2 (S), R43.2, TP20.1
- no-connect marks 0 -> 2
Other:
- note added: "Q Estimate"
- note removed: "Q Estimate Circuit"

Commit message: pushing
Parts:
- added C55: 0.1u, symbol Device:C
- added C56: 1u, symbol Device:C
- added C9: 10p, symbol Device:C
- added R10: 0, symbol Device:R
- added TP22: ASK_TST, symbol Connector:TestPoint_Probe
Connections:
- net VBB_1 is gone; now on net IOUT_CSN_0: C29.1, C30.1, C31.1, C32.1, Q4.5 (DRAIN), Q4.6 (DRAIN), Q4.7 (DRAIN), Q4.8 (DRAIN), Q6.5 (DRAIN), Q6.6 (DRAIN), Q6.7 (DRAIN), Q6.8 (DRAIN), R23.2, R28.1
- net BST2_1: now also U1.43 (BST2_1)
- net GND: now also U1.49 (PGND_1), C55.1, C56.1, C9.2
- net HG2_1: now also U1.44 (HG2_1)
- net LG2_1: now also U1.47 (LG2_1)
- net SW2_1: now also U1.45 (SW2_1)
- net VDDD: now also U1.48 (PVDD_1), C55.2, C56.2
- net at U1.42 (ASK_TST): now also R10.1
- net IOUT_CSN_0: now reaches U1.46 (VBB_1)
- new net: C9.1, R10.2, TP22.1

Commit message: starting pcb
Parts:
- added C57: 0.1u, symbol Device:C
- added C58: 1u, symbol Device:C
Connections:
- net BST1_1: now also U1.53 (BST1_1)
- net GND: now also U1.3 (PGND_0), C57.1, C58.1
- net HG1_1: now also U1.52 (HG1_1)
- net LG1_0: now also U1.2 (LG1_0)
- net LG1_1: now also U1.50 (LG1_1)
- net Q_COMP: now also U1.32 (QCOMP2)
- net SW1_0: now also U1.1 (SW1_0)
- net SW1_1: now also U1.51 (SW1_1)
- net VDDD: now also U1.4 (PVDD_0), C57.2, C58.2
- net QComp: no longer names the net of U1.37 (QCOMP1)
- net QComp: no longer U1.32 (QCOMP2)
- net VDDD_in: no longer names the net of C44.2, C45.2, R26.2, TP17.1, U1.63 (VDDD)
- no-connect marks 2 -> 8
Other:
- moved on the sheet: C42, C43, C44, C45, C53, C54, R25, R26, TP16, TP17
