File: project.kicad_sch (KiCad schematic)
At the start: 150 parts, among them J1 Conn_01x02_Pin, J3 Conn_01x01_Pin, J4 Conn_01x05_Socket, Q1 BSZ0902NS, Q2 BSZ0902NS, Q3 BSZ0902NS, Q4 BSZ0902NS, Q5 BSZ0902NS, Q6 BSZ0902NS, Q7 BSZ0902NS, Q8 BSS138N, U1 WLC1115-68LQXQ, U2 SLS32AIA020U2USON10XTMA1, U3 LMV358AQDGKRQ1

Commit message: codex
Parts:
- C1, C10, C11, C12, C13, C14, C15, C16, C17, C18, C19, C2, C20, C21, C22, C23, C24, C25, C26, C27, C28, C29, C3, C30, C31, C32, C33, C34, C35, C36, C37, C38, C39, C40, C41, C42, C43, C44, C45, C46, C47, C48, C49, C5, C50, C51, C52, C53, C54, C55, C56, C57, C58, C6, C7, C8, C9: footprint (none) -> Capacitor_SMD:C_0603_1608Metric_Pad1.08x0.95mm_HandSolder
- C4: value 0.47n -> 0.47u; footprint (none) -> Capacitor_SMD:C_0603_1608Metric_Pad1.08x0.95mm_HandSolder
- D1, D2: footprint (none) -> LED_SMD:LED_0201_0603Metric_Pad0.64x0.40mm_HandSolder
- D10, D11, D8, D9: footprint RB511SM40FHT2R -> rb511sm:RB511SM40FHT2R
- D12: footprint SOD3716X135N -> 1N4448W-TP:SOD3716X135N
- D13: footprint SOT95P240X120-3N -> MMBD1503A:SOT95P240X120-3N
- D5, D6: value Diode -> bat54s; footprint (none) -> bat54s:P200_SOT-23
- D7: footprint SODFL1608X65N -> bat64t5q:SODFL1608X65N
- J1: footprint (none) -> Connector_PinHeader_2.54mm:PinHeader_1x02_P2.54mm_Vertical
- J3: footprint (none) -> Connector_PinHeader_2.54mm:PinHeader_1x01_P2.54mm_Vertical
- J4: footprint (none) -> Connector_PinHeader_2.54mm:PinHeader_1x05_P2.54mm_Vertical
- L2: footprint (none) -> TerminalBlock_Phoenix:TerminalBlock_Phoenix_MKDS-1,5-2-5.08_1x02_P5.08mm_Horizontal
- Q2, Q3, Q4, Q5, Q6, Q7: footprint (none) -> NFET:IFX-PG-TSDSON-8-26-V
- R1, R10, R11, R12, R13, R14, R15, R16, R17, R18, R19, R2, R20, R21, R22, R23, R24, R25, R26, R27, R28, R29, R3, R30, R31, R32, R33, R34, R35, R36, R37, R38, R39, R4, R40, R41, R42, R43, R5, R6, R7, R8, R9: footprint (none) -> Resistor_SMD:R_0603_1608Metric_Pad0.98x0.95mm_HandSolder
- TP1, TP10, TP11, TP12, TP13, TP14, TP15, TP16, TP17, TP18, TP19, TP2, TP20, TP21, TP22, TP3, TP4, TP5, TP6, TP7, TP8, TP9: footprint (none) -> TestPoint:TestPoint_Pad_D2.0mm
- U1: footprint PG-VQFN-68 -> wlc1115:PG-VQFN-68
- U2: footprint PG-USON-10-2 -> optigatrust:PG-USON-10-2
- U3: footprint DGK8_TEX -> opamp:DGK8_TEX
Connections:
- net GND: now also D13.1 (ANODE), U2.11 (EPAD); no longer D13.2 (CATHODE)
- net Q_COMP: now also U1.37 (QCOMP1)
- net VDDD: now also D13.2 (CATHODE); no longer D13.1 (ANODE)

Commit message: idk what im doing
Parts:
- L1: footprint ProtoFlow.pretty:Yageo_Pulse_PA4342_10.3x11.5mm -> PA4342.682NLT:Yageo_Pulse_PA4342_10.3x11.5mm
Changed lines of the file:
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@@
 			)
 		)
-		(property "Footprint" "ProtoFlow.pretty:Yageo_Pulse_PA4342_10.3x11.5mm"
+		(property "Footprint" "PA4342.682NLT:Yageo_Pulse_PA4342_10.3x11.5mm"
 			(at 325.12 204.47 0)
 			(hide yes)

Commit message: bro
Parts:
- removed D5, D6: bat54s, bat54s:P200_SOT-23, symbol bat54s:Diode-NC_pin
- removed Q1: BSZ0902NS, NFET:IFX-PG-TSDSON-8-26-V, symbol NFET:BSZ0902NS
- removed R26: 0, Resistor_SMD:R_0603_1608Metric_Pad0.98x0.95mm_HandSolder, symbol Device:R
- added IC1: BAT5404WH6327XTSA1, bat54sdual:SOT65P210X100-3N, symbol bat54dual:BAT5404WH6327XTSA1
- added J2: Conn_01x02_Pin, Connector_PinHeader_2.54mm:PinHeader_1x02_P2.54mm_Horizontal, symbol Connector:Conn_01x02_Pin
- added J5: Conn_01x02, Connector_Wire:SolderWire-0.5sqmm_1x02_P4.8mm_D0.9mm_OD2.3mm, symbol Connector_Generic:Conn_01x02
- added TP23: VCCD, TestPoint:TestPoint_Pad_D1.0mm, symbol Connector:TestPoint_Probe
- C20, C21, C23, C24, C25, C26, C34, C35, C36, C37, C38: footprint Capacitor_SMD:C_0603_1608Metric_Pad1.08x0.95mm_HandSolder -> Capacitor_SMD:C_1206_3216Metric_Pad1.33x1.80mm_HandSolder
- C22, C39, C47, C53, C54, C55, C56, C57, C58, C9: footprint Capacitor_SMD:C_0603_1608Metric_Pad1.08x0.95mm_HandSolder -> Capacitor_SMD:C_0402_1005Metric_Pad0.74x0.62mm_HandSolder
- C27, C29, C44: footprint Capacitor_SMD:C_0603_1608Metric_Pad1.08x0.95mm_HandSolder -> Capacitor_SMD:C_0805_2012Metric_Pad1.18x1.45mm_HandSolder
- C8: footprint Capacitor_SMD:C_0603_1608Metric_Pad1.08x0.95mm_HandSolder -> Resistor_SMD:R_0402_1005Metric_Pad0.72x0.64mm_HandSolder
- D10, D11, D8, D9: footprint rb511sm:RB511SM40FHT2R -> Diode_SMD:D_SOD-523
- J1: footprint Connector_PinHeader_2.54mm:PinHeader_1x02_P2.54mm_Vertical -> Connector_PinHeader_2.54mm:PinHeader_1x02_P2.54mm_Horizontal
- J3: footprint Connector_PinHeader_2.54mm:PinHeader_1x01_P2.54mm_Vertical -> Connector_PinHeader_2.54mm:PinHeader_1x02_P2.54mm_Horizontal
- J4: footprint Connector_PinHeader_2.54mm:PinHeader_1x05_P2.54mm_Vertical -> Connector_PinHeader_2.54mm:PinHeader_1x05_P2.54mm_Horizontal
- R10, R27, R28, R30, R8, R9: footprint Resistor_SMD:R_0603_1608Metric_Pad0.98x0.95mm_HandSolder -> Resistor_SMD:R_0402_1005Metric_Pad0.72x0.64mm_HandSolder
- R22, R23: footprint Resistor_SMD:R_0603_1608Metric_Pad0.98x0.95mm_HandSolder -> Resistor_SMD:R_1206_3216Metric_Pad1.30x1.75mm_HandSolder
- R43: footprint Resistor_SMD:R_0603_1608Metric_Pad0.98x0.95mm_HandSolder -> Capacitor_SMD:C_0402_1005Metric_Pad0.74x0.62mm_HandSolder
- TP1: value TestPoint_Probe -> ASK_OUT; footprint TestPoint:TestPoint_Pad_D2.0mm -> TestPoint:TestPoint_Pad_D1.5mm
- TP16, TP17, TP8: footprint TestPoint:TestPoint_Pad_D2.0mm -> TestPoint:TestPoint_Pad_D1.5mm
- TP22: footprint TestPoint:TestPoint_Pad_D2.0mm -> TestPoint:TestPoint_Pad_D1.0mm
Connections:
- net GND: now also D1.1 (K), D2.1 (K), J4.2 (Pin_2), J5.2 (Pin_2); no longer J4.4 (Pin_4), R6.1, R7.1
- net HPI_I2C_SCL: now also J4.4 (Pin_4); no longer J4.2 (Pin_2)
- net HPI_I2C_SDA: now also J4.5 (Pin_5); no longer J4.1 (Pin_1)
- net IOUT_CSP_0: now also R9.2; no longer R9.1
- net PVIN_0: now also J5.1 (Pin_1)
- net VDDD: now also C44.2, C45.2, TP17.1, U1.63 (VDDD)
- net XRES: now also J2.2 (Pin_2)
- net toESP: now also J2.1 (Pin_1)
- net at R7.2: now also U1.27 (LED2); no longer D2.1 (K)
- net at U1.26 (LED1): now also R6.2; no longer D1.2 (A)
- net at D2.2 (A): now also R7.1; no longer U1.27 (LED2)
- net at U1.6 (VBB_0): now also R9.1; no longer R9.2
- net at C1.1, U1.62 (VCCD): now also TP23.1
- net at C12.1, R12.2, R14.1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: now also IC1.3 (A/K)
- net at C19.1, D7.2 (A): now also J4.1 (Pin_1); no longer J4.5 (Pin_5)
- net at C11.2, R13.1: now also IC1.1 (A), IC1.2 (K)
- net NFet Control: no longer names the net of U1.35 (NFET_CTRL_1)
- new net: D1.2 (A), R6.1
- no-connect marks 8 -> 10
Other:
- moved on the sheet: D1, D2, J4, R6, R7, R9

Commit message: before work
Parts:
- removed R4: 1k, Resistor_SMD:R_0603_1608Metric_Pad0.98x0.95mm_HandSolder, symbol Device:R
- removed R5: 2k, Resistor_SMD:R_0603_1608Metric_Pad0.98x0.95mm_HandSolder, symbol Device:R
- TP10, TP21, TP6, TP7, TP9: footprint TestPoint:TestPoint_Pad_D2.0mm -> TestPoint:TestPoint_Pad_D1.0mm
Other:
- note removed: "IC -> ESP"
