File: project.kicad_sch (KiCad schematic)
At the start: 148 parts, among them IC1 BAT5404WH6327XTSA1, J1 Conn_01x02_Pin, J2 Conn_01x02_Pin, J3 Conn_01x01_Pin, J4 Conn_01x05_Socket, J5 Conn_01x02, Q2 BSZ0902NS, Q3 BSZ0902NS, Q4 BSZ0902NS, Q5 BSZ0902NS, Q6 BSZ0902NS, Q7 BSZ0902NS, Q8 BSS138N, U1 WLC1115-68LQXQ, U2 SLS32AIA020U2USON10XTMA1, U3 LMV358AQDGKRQ1

Commit message: should be actaully done now brah
Parts:
- added H1, H2, H3, H4: MountingHole, MountingHole:MountingHole_3.2mm_M3_Pad, symbol Mechanical:MountingHole
- C8: footprint Resistor_SMD:R_0402_1005Metric_Pad0.72x0.64mm_HandSolder -> Capacitor_SMD:C_0402_1005Metric_Pad0.74x0.62mm_HandSolder
- J3: footprint Connector_PinHeader_2.54mm:PinHeader_1x02_P2.54mm_Horizontal -> Connector_PinHeader_2.54mm:PinHeader_1x01_P2.54mm_Horizontal
- R43: footprint Capacitor_SMD:C_0402_1005Metric_Pad0.74x0.62mm_HandSolder -> Resistor_SMD:R_0402_1005Metric_Pad0.72x0.64mm_HandSolder
Other:
- note removed: "Power NFet"
