File: project.kicad_pcb (KiCad board)
At the start: 2 copper layers, 2 parts, among them Q1 BSZ0902NS, Q8 BSS138N

Commit message: codex
Parts:
- added C1: 0.1u, Capacitor_SMD:C_0603_1608Metric_Pad1.08x0.95mm_HandSolder, F.Cu at (52.0, 73.2)
- added C10: 22nf, Capacitor_SMD:C_0603_1608Metric_Pad1.08x0.95mm_HandSolder, F.Cu at (27.0, 102.0)
- added C11: 0.22uf, Capacitor_SMD:C_0603_1608Metric_Pad1.08x0.95mm_HandSolder, F.Cu at (30.8, 101.2)
- added C12: 22n, Capacitor_SMD:C_0603_1608Metric_Pad1.08x0.95mm_HandSolder, F.Cu at (32.0, 103.0)
- added C13: 0.1u, Capacitor_SMD:C_0603_1608Metric_Pad1.08x0.95mm_HandSolder, F.Cu at (40.0, 95.2)
- added C14: 330p, Capacitor_SMD:C_0603_1608Metric_Pad1.08x0.95mm_HandSolder, F.Cu at (38.8, 89.8)
- added C15: 150p, Capacitor_SMD:C_0603_1608Metric_Pad1.08x0.95mm_HandSolder, F.Cu at (42.5, 91.2)
- added C16: 10n, Capacitor_SMD:C_0603_1608Metric_Pad1.08x0.95mm_HandSolder, F.Cu at (37.8, 99.5)
- added C17: 0.1u, Capacitor_SMD:C_0603_1608Metric_Pad1.08x0.95mm_HandSolder, F.Cu at (49.5, 88.0)
- added C18: 1u, Capacitor_SMD:C_0603_1608Metric_Pad1.08x0.95mm_HandSolder, F.Cu at (56.2, 90.2)
- added C19: 0.1u, Capacitor_SMD:C_0603_1608Metric_Pad1.08x0.95mm_HandSolder, F.Cu at (56.2, 107.8)
- added C2: 2.2u, Capacitor_SMD:C_0603_1608Metric_Pad1.08x0.95mm_HandSolder, F.Cu at (45.0, 83.0)
- added C20: 22u, Capacitor_SMD:C_0603_1608Metric_Pad1.08x0.95mm_HandSolder, F.Cu at (28.5, 53.0)
- added C21: 22u, Capacitor_SMD:C_0603_1608Metric_Pad1.08x0.95mm_HandSolder, F.Cu at (32.2, 52.2)
- added C22: 0.1u, Capacitor_SMD:C_0603_1608Metric_Pad1.08x0.95mm_HandSolder, F.Cu at (47.0, 72.2)
- added C23: 22u, Capacitor_SMD:C_0603_1608Metric_Pad1.08x0.95mm_HandSolder, F.Cu at (58.0, 52.5)
- added C24: 22u, Capacitor_SMD:C_0603_1608Metric_Pad1.08x0.95mm_HandSolder, F.Cu at (61.8, 51.8)
- added C25: 22u, Capacitor_SMD:C_0603_1608Metric_Pad1.08x0.95mm_HandSolder, F.Cu at (58.0, 66.5)
- added C26: 22u, Capacitor_SMD:C_0603_1608Metric_Pad1.08x0.95mm_HandSolder, F.Cu at (61.8, 65.8)
- added C27: 4.7u, Capacitor_SMD:C_0603_1608Metric_Pad1.08x0.95mm_HandSolder, F.Cu at (30.2, 56.2)
- added C28: 10n, Capacitor_SMD:C_0603_1608Metric_Pad1.08x0.95mm_HandSolder, F.Cu at (30.5, 59.0)
- added C29: 22u, Capacitor_SMD:C_0603_1608Metric_Pad1.08x0.95mm_HandSolder, F.Cu at (69.0, 64.0)
- added C3: 1n, Capacitor_SMD:C_0603_1608Metric_Pad1.08x0.95mm_HandSolder, F.Cu at (45.2, 76.8)
- added C30: 22u, Capacitor_SMD:C_0603_1608Metric_Pad1.08x0.95mm_HandSolder, F.Cu at (72.8, 63.2)
- added C31: 0.1u, Capacitor_SMD:C_0603_1608Metric_Pad1.08x0.95mm_HandSolder, F.Cu at (69.0, 78.0)
- added C32: 0.1u, Capacitor_SMD:C_0603_1608Metric_Pad1.08x0.95mm_HandSolder, F.Cu at (72.8, 77.2)
- added C33: 10n, Capacitor_SMD:C_0603_1608Metric_Pad1.08x0.95mm_HandSolder, F.Cu at (83.0, 73.0)
- added C34: 0.1u, Capacitor_SMD:C_0603_1608Metric_Pad1.08x0.95mm_HandSolder, F.Cu at (77.0, 92.0)
- added C35: 0.1u, Capacitor_SMD:C_0603_1608Metric_Pad1.08x0.95mm_HandSolder, F.Cu at (76.5, 94.5)
- added C36: 0.1u, Capacitor_SMD:C_0603_1608Metric_Pad1.08x0.95mm_HandSolder, F.Cu at (76.5, 97.5)
- added C37: 0.1u, Capacitor_SMD:C_0603_1608Metric_Pad1.08x0.95mm_HandSolder, F.Cu at (76.5, 100.5)
- added C38: 0.1u, Capacitor_SMD:C_0603_1608Metric_Pad1.08x0.95mm_HandSolder, F.Cu at (76.5, 103.5)
- added C39: 0.1u, Capacitor_SMD:C_0603_1608Metric_Pad1.08x0.95mm_HandSolder, F.Cu at (59.0, 77.0)
- added C4: 0.47u, Capacitor_SMD:C_0603_1608Metric_Pad1.08x0.95mm_HandSolder, F.Cu at (39.0, 77.0)
- added C40: 0.1u, Capacitor_SMD:C_0603_1608Metric_Pad1.08x0.95mm_HandSolder, F.Cu at (59.8, 71.5)
- added C41: 10n, Capacitor_SMD:C_0603_1608Metric_Pad1.08x0.95mm_HandSolder, F.Cu at (83.0, 85.0)
- added C42: 1u, Capacitor_SMD:C_0603_1608Metric_Pad1.08x0.95mm_HandSolder, F.Cu at (50.8, 68.8)
- added C43: 0.1u, Capacitor_SMD:C_0603_1608Metric_Pad1.08x0.95mm_HandSolder, F.Cu at (50.8, 71.5)
- added C44: 1u, Capacitor_SMD:C_0603_1608Metric_Pad1.08x0.95mm_HandSolder, F.Cu at (56.0, 69.5)
- added C45: 0.1u, Capacitor_SMD:C_0603_1608Metric_Pad1.08x0.95mm_HandSolder, F.Cu at (56.0, 72.2)
- added C46: 10n, Capacitor_SMD:C_0603_1608Metric_Pad1.08x0.95mm_HandSolder, F.Cu at (61.0, 88.0)
- added C47: 470n, Capacitor_SMD:C_0603_1608Metric_Pad1.08x0.95mm_HandSolder, F.Cu at (64.8, 87.2)
- added C48: 10n, Capacitor_SMD:C_0603_1608Metric_Pad1.08x0.95mm_HandSolder, F.Cu at (66.0, 89.0)
- added C49: 0.1u, Capacitor_SMD:C_0603_1608Metric_Pad1.08x0.95mm_HandSolder, F.Cu at (61.0, 97.0)
- added C5: 0.1u, Capacitor_SMD:C_0603_1608Metric_Pad1.08x0.95mm_HandSolder, F.Cu at (49.0, 94.0)
- added C50: 100n, Capacitor_SMD:C_0603_1608Metric_Pad1.08x0.95mm_HandSolder, F.Cu at (64.8, 96.2)
- added C51: 5.6n, Capacitor_SMD:C_0603_1608Metric_Pad1.08x0.95mm_HandSolder, F.Cu at (61.0, 100.0)
- added C52: 1n, Capacitor_SMD:C_0603_1608Metric_Pad1.08x0.95mm_HandSolder, F.Cu at (72.0, 103.0)
- added C53: 0.1u, Capacitor_SMD:C_0603_1608Metric_Pad1.08x0.95mm_HandSolder, F.Cu at (59.0, 81.0)
- added C54: 0.1u, Capacitor_SMD:C_0603_1608Metric_Pad1.08x0.95mm_HandSolder, F.Cu at (61.5, 81.5)
- added C55: 0.1u, Capacitor_SMD:C_0603_1608Metric_Pad1.08x0.95mm_HandSolder, F.Cu at (49.0, 86.0)
- added C56: 1u, Capacitor_SMD:C_0603_1608Metric_Pad1.08x0.95mm_HandSolder, F.Cu at (52.8, 85.2)
- added C57: 0.1u, Capacitor_SMD:C_0603_1608Metric_Pad1.08x0.95mm_HandSolder, F.Cu at (54.0, 87.0)
- added C58: 1u, Capacitor_SMD:C_0603_1608Metric_Pad1.08x0.95mm_HandSolder, F.Cu at (57.8, 86.2)
- added C6: 1u, Capacitor_SMD:C_0603_1608Metric_Pad1.08x0.95mm_HandSolder, F.Cu at (55.0, 94.0)
- added C7: 0.1u, Capacitor_SMD:C_0603_1608Metric_Pad1.08x0.95mm_HandSolder, F.Cu at (45.8, 87.8)
- added C8: 0.1u, Capacitor_SMD:C_0603_1608Metric_Pad1.08x0.95mm_HandSolder, F.Cu at (45.8, 89.5)
- added C9: 10p, Capacitor_SMD:C_0603_1608Metric_Pad1.08x0.95mm_HandSolder, F.Cu at (59.0, 84.5)
- added D1: LED, LED_SMD:LED_0201_0603Metric_Pad0.64x0.40mm_HandSolder, F.Cu at (32.0, 109.0)
- added D10: RB511SM-40FHT2R, rb511sm:RB511SM40FHT2R, F.Cu at (62.2, 76.8)
- added D11: RB511SM-40FHT2R, rb511sm:RB511SM40FHT2R, F.Cu at (64.0, 70.5)
- added D12: 1N4448W-TP, 1N4448W-TP:SOD3716X135N, F.Cu at (68.0, 104.0)
- added D13: MMBD1503A, MMBD1503A:SOT95P240X120-3N, F.Cu at (62.0, 103.0)
- added D2: LED, LED_SMD:LED_0201_0603Metric_Pad0.64x0.40mm_HandSolder, F.Cu at (38.0, 109.0)
- added D5: bat54s, bat54s:P200_SOT-23, F.Cu at (25.5, 90.0)
- added D6: bat54s, bat54s:P200_SOT-23, F.Cu at (25.5, 96.0)
- added D7: BAT64T5Q-7-F, bat64t5q:SODFL1608X65N, F.Cu at (53.0, 108.0)
- added D8: RB511SM-40FHT2R, rb511sm:RB511SM40FHT2R, F.Cu at (43.0, 70.5)
- added D9: RB511SM-40FHT2R, rb511sm:RB511SM40FHT2R, F.Cu at (42.8, 75.2)
- added FID1: Fiducial_1mm_Mask2mm, Fiducial_1mm_Mask2mm, F.Cu at (20.5, 50.5)
- added FID2: Fiducial_1mm_Mask2mm, Fiducial_1mm_Mask2mm, F.Cu at (89.5, 50.5)
- added FID3: Fiducial_1mm_Mask2mm, Fiducial_1mm_Mask2mm, F.Cu at (89.5, 114.5)
- added J1: Conn_01x02_Pin, Connector_PinHeader_2.54mm:PinHeader_1x02_P2.54mm_Vertical, F.Cu at (23.0, 108.5)
- added J3: Conn_01x01_Pin, Connector_PinHeader_2.54mm:PinHeader_1x01_P2.54mm_Vertical, F.Cu at (88.0, 110.0)
- added J4: Conn_01x05_Socket, Connector_PinHeader_2.54mm:PinHeader_1x05_P2.54mm_Vertical, F.Cu at (49.0, 112.0)
- added L1: PA4342.682NLT, ProtoFlow.pretty:Yageo_Pulse_PA4342_10.3x11.5mm, F.Cu at (49.5, 59.5)
- added L2: MP-A11, TerminalBlock_Phoenix:TerminalBlock_Phoenix_MKDS-1,5-2-5.08_1x02_P5.08mm_Horizontal, F.Cu at (84.3, 101.5)
- added Q2: BSZ0902NS, NFET:IFX-PG-TSDSON-8-26-V, F.Cu at (37.5, 57.5)
- added Q3: BSZ0902NS, NFET:IFX-PG-TSDSON-8-26-V, F.Cu at (37.5, 62.0)
- added Q4: BSZ0902NS, NFET:IFX-PG-TSDSON-8-26-V, F.Cu at (78.5, 67.0)
- added Q5: BSZ0902NS, NFET:IFX-PG-TSDSON-8-26-V, F.Cu at (78.5, 72.0)
- added Q6: BSZ0902NS, NFET:IFX-PG-TSDSON-8-26-V, F.Cu at (78.5, 79.0)
- added Q7: BSZ0902NS, NFET:IFX-PG-TSDSON-8-26-V, F.Cu at (78.5, 84.0)
- added R1: 1k, Resistor_SMD:R_0603_1608Metric_Pad0.98x0.95mm_HandSolder, F.Cu at (40.8, 79.5)
- added R10: 0, Resistor_SMD:R_0603_1608Metric_Pad0.98x0.95mm_HandSolder, F.Cu at (62.8, 85.2)
- added R11: 1k, Resistor_SMD:R_0603_1608Metric_Pad0.98x0.95mm_HandSolder, F.Cu at (35.8, 102.2)
- added R12: 27k, Resistor_SMD:R_0603_1608Metric_Pad0.98x0.95mm_HandSolder, F.Cu at (29.0, 87.5)
- added R13: 5.1k, Resistor_SMD:R_0603_1608Metric_Pad0.98x0.95mm_HandSolder, F.Cu at (29.8, 90.8)
- added R14: 390, Resistor_SMD:R_0603_1608Metric_Pad0.98x0.95mm_HandSolder, F.Cu at (29.8, 95.8)
- added R15: 10k, Resistor_SMD:R_0603_1608Metric_Pad0.98x0.95mm_HandSolder, F.Cu at (38.2, 95.8)
- added R16: 100k, Resistor_SMD:R_0603_1608Metric_Pad0.98x0.95mm_HandSolder, F.Cu at (35.0, 89.0)
- added R17: 0, Resistor_SMD:R_0603_1608Metric_Pad0.98x0.95mm_HandSolder, F.Cu at (35.0, 99.0)
- added R18: 1M, Resistor_SMD:R_0603_1608Metric_Pad0.98x0.95mm_HandSolder, F.Cu at (40.0, 99.0)
- added R19: 10k, Resistor_SMD:R_0603_1608Metric_Pad0.98x0.95mm_HandSolder, F.Cu at (57.8, 93.0)
- added R2: 5.1k, Resistor_SMD:R_0603_1608Metric_Pad0.98x0.95mm_HandSolder, F.Cu at (54.0, 105.0)
- added R20: 5.1k, Resistor_SMD:R_0603_1608Metric_Pad0.98x0.95mm_HandSolder, F.Cu at (53.2, 96.8)
- added R21: 5.1k, Resistor_SMD:R_0603_1608Metric_Pad0.98x0.95mm_HandSolder, F.Cu at (56.2, 96.8)
- added R22: 0.005, Resistor_SMD:R_0603_1608Metric_Pad0.98x0.95mm_HandSolder, F.Cu at (33.0, 56.0)
- added R23: 0.01, Resistor_SMD:R_0603_1608Metric_Pad0.98x0.95mm_HandSolder, F.Cu at (59.0, 59.5)
- added R24: 0, Resistor_SMD:R_0603_1608Metric_Pad0.98x0.95mm_HandSolder, F.Cu at (86.0, 85.0)
- added R25: 0, Resistor_SMD:R_0603_1608Metric_Pad0.98x0.95mm_HandSolder, F.Cu at (47.0, 69.5)
- added R26: 0, Resistor_SMD:R_0603_1608Metric_Pad0.98x0.95mm_HandSolder, F.Cu at (59.8, 68.8)
- added R27: 10, Resistor_SMD:R_0603_1608Metric_Pad0.98x0.95mm_HandSolder, F.Cu at (41.8, 82.2)
- added R28: 10, Resistor_SMD:R_0603_1608Metric_Pad0.98x0.95mm_HandSolder, F.Cu at (42.0, 84.0)
- added R29: 0, Resistor_SMD:R_0603_1608Metric_Pad0.98x0.95mm_HandSolder, F.Cu at (42.0, 86.0)
- added R3: 0, Resistor_SMD:R_0603_1608Metric_Pad0.98x0.95mm_HandSolder, F.Cu at (86.0, 73.0)
- added R30: 0, Resistor_SMD:R_0603_1608Metric_Pad0.98x0.95mm_HandSolder, F.Cu at (42.0, 88.0)
- added R31: 5.1k, Resistor_SMD:R_0603_1608Metric_Pad0.98x0.95mm_HandSolder, F.Cu at (57.8, 104.2)
- added R32: 10, Resistor_SMD:R_0603_1608Metric_Pad0.98x0.95mm_HandSolder, F.Cu at (61.0, 91.0)
- added R33: 10, Resistor_SMD:R_0603_1608Metric_Pad0.98x0.95mm_HandSolder, F.Cu at (68.5, 92.5)
- added R34: 62, Resistor_SMD:R_0603_1608Metric_Pad0.98x0.95mm_HandSolder, F.Cu at (64.8, 91.8)
- added R35: 2.2k, Resistor_SMD:R_0603_1608Metric_Pad0.98x0.95mm_HandSolder, F.Cu at (61.0, 94.0)
- added R36: 130k, Resistor_SMD:R_0603_1608Metric_Pad0.98x0.95mm_HandSolder, F.Cu at (66.8, 94.2)
- added R37: 0, Resistor_SMD:R_0603_1608Metric_Pad0.98x0.95mm_HandSolder, F.Cu at (66.0, 98.0)
- added R38: 100k, Resistor_SMD:R_0603_1608Metric_Pad0.98x0.95mm_HandSolder, F.Cu at (67.0, 100.0)
- added R39: 5.1k, Resistor_SMD:R_0603_1608Metric_Pad0.98x0.95mm_HandSolder, F.Cu at (72.0, 106.8)
- added R4: 1k, Resistor_SMD:R_0603_1608Metric_Pad0.98x0.95mm_HandSolder, F.Cu at (28.0, 106.0)
- added R40: 36k, Resistor_SMD:R_0603_1608Metric_Pad0.98x0.95mm_HandSolder, F.Cu at (65.0, 103.0)
- added R41: 3.6k, Resistor_SMD:R_0603_1608Metric_Pad0.98x0.95mm_HandSolder, F.Cu at (65.0, 106.8)
- added R42: 20k, Resistor_SMD:R_0603_1608Metric_Pad0.98x0.95mm_HandSolder, F.Cu at (61.0, 107.0)
- added R43: 0, Resistor_SMD:R_0603_1608Metric_Pad0.98x0.95mm_HandSolder, F.Cu at (63.2, 108.2)
- added R5: 2k, Resistor_SMD:R_0603_1608Metric_Pad0.98x0.95mm_HandSolder, F.Cu at (28.0, 109.0)
- added R6: 1k, Resistor_SMD:R_0603_1608Metric_Pad0.98x0.95mm_HandSolder, F.Cu at (35.0, 109.0)
- added R7: 1k, Resistor_SMD:R_0603_1608Metric_Pad0.98x0.95mm_HandSolder, F.Cu at (41.0, 109.0)
- added R8: 0, Resistor_SMD:R_0603_1608Metric_Pad0.98x0.95mm_HandSolder, F.Cu at (39.0, 72.5)
- added R9: 0, Resistor_SMD:R_0603_1608Metric_Pad0.98x0.95mm_HandSolder, F.Cu at (37.2, 73.2)
- added TP1: TestPoint_Probe, TestPoint:TestPoint_Pad_D2.0mm, F.Cu at (22.0, 83.5)
- added TP10: LG2_1, TestPoint:TestPoint_Pad_D2.0mm, F.Cu at (88.0, 61.5)
- added TP11: COIL_SNS, TestPoint:TestPoint_Pad_D2.0mm, F.Cu at (82.5, 88.5)
- added TP12: HG1_1, TestPoint:TestPoint_Pad_D2.0mm, F.Cu at (88.0, 69.5)
- added TP13: LG1_1, TestPoint:TestPoint_Pad_D2.0mm, F.Cu at (86.0, 76.5)
- added TP14: SW2_1, TestPoint:TestPoint_Pad_D2.0mm, F.Cu at (88.0, 65.5)
- added TP15: SW1_1, TestPoint:TestPoint_Pad_D2.0mm, F.Cu at (86.5, 80.0)
- added TP16: Vin, TestPoint:TestPoint_Pad_D2.0mm, F.Cu at (26.8, 111.8)
- added TP17: VDDD, TestPoint:TestPoint_Pad_D2.0mm, F.Cu at (86.0, 88.5)
- added TP18: VBRG_0, TestPoint:TestPoint_Pad_D2.0mm, F.Cu at (83.0, 80.0)
- added TP19: V2I_IP, TestPoint:TestPoint_Pad_D2.0mm, F.Cu at (74.0, 112.0)
- added TP2: OPAMP_GAIN, TestPoint:TestPoint_Pad_D2.0mm, F.Cu at (22.0, 87.5)
- added TP20: Q_COMP, TestPoint:TestPoint_Pad_D2.0mm, F.Cu at (82.0, 112.0)
- added TP21: PWN_OUT, TestPoint:TestPoint_Pad_D2.0mm, F.Cu at (22.0, 99.5)
- added TP22: ASK_TST, TestPoint:TestPoint_Pad_D2.0mm, F.Cu at (22.0, 103.5)
- added TP3: OPAMP_CMP, TestPoint:TestPoint_Pad_D2.0mm, F.Cu at (22.0, 91.5)
- added TP4: CMP_REF, TestPoint:TestPoint_Pad_D2.0mm, F.Cu at (22.0, 95.5)
- added TP5: PVIN_0, TestPoint:TestPoint_Pad_D2.0mm, F.Cu at (22.0, 53.5)
- added TP6: HG1_0, TestPoint:TestPoint_Pad_D2.0mm, F.Cu at (22.0, 57.5)
- added TP7: LG1_0, TestPoint:TestPoint_Pad_D2.0mm, F.Cu at (22.0, 61.5)
- added TP8: SW1_0, TestPoint:TestPoint_Pad_D2.0mm, F.Cu at (22.0, 65.5)
- added TP9: HG2_1, TestPoint:TestPoint_Pad_D2.0mm, F.Cu at (88.0, 57.5)
- added U1: WLC1115-68LQXQ, wlc1115:PG-VQFN-68, F.Cu at (52.0, 79.0)
- added U2: SLS32AIA020U2USON10XTMA1, optigatrust:PG-USON-10-2, F.Cu at (52.0, 91.0)
- added U3: LMV358AQDGKRQ1, opamp:DGK8_TEX, F.Cu at (34.0, 94.0)
- moved Q1 133.2 mm to (24.5, 68.0), turned to -90 degrees
- moved Q8 95.1 mm to (69.0, 109.0)
Routing:
- net GND: track 0.00 -> 493.9 mm, vias 0 -> 25
- net VDDD: track 0.00 -> 218.9 mm, vias 0 -> 7
- net /IOUT_CSN_0: track 0.00 -> 116.2 mm, vias 0 -> 4
- net /IOUT_CSP_0: track 0.00 -> 96.2 mm, vias 0 -> 8
- net PVIN_0: track 0.00 -> 89.5 mm, vias 0 -> 2
- net /SW2_1: track 0.00 -> 85.7 mm, vias 0 -> 3
- net Net-(C9-Pad1): track 0.00 -> 84.1 mm, vias 0 -> 2
- net /SW1_1: track 0.00 -> 73.9 mm
- net /ASK_DEMOD: track 0.00 -> 72.4 mm, vias 0 -> 3
- net Net-(J1-Pin_1): track 0.00 -> 69.9 mm, vias 0 -> 1
- net /Vin: track 0.00 -> 65.2 mm, vias 0 -> 3
- net /NFet Control: track 0.00 -> 62.6 mm, vias 0 -> 2
- net Net-(C44-Pad2): track 0.00 -> 62.3 mm, vias 0 -> 2
- net /ASK_OUT: track 0.00 -> 59.2 mm, vias 0 -> 2
- net /SW1_0: track 0.00 -> 58.3 mm
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- added copper zone on F.Cu, net /COIL_SNS
- added copper zone on F.Cu, net /IIN_CSN_0
- added copper zone on F.Cu, net /IOUT_CSN_0
- added copper zone on F.Cu, net /IOUT_CSP_0
- added copper zone on F.Cu, net /SW1_0
- added copper zone on F.Cu, net /SW1_1
- added copper zone on F.Cu, net /SW2_1
- added copper zone on B.Cu, net GND
- added copper zone on F.Cu, net GND
- added copper zone on F.Cu, net PVIN_0
Other:
- board outline added: 74 x 69 mm

Commit message: idk
Routing:
- net GND: track 493.9 -> 297.7 mm
- net /Vin: track 65.2 -> 64.7 mm

Commit message: idk what im doing
Parts:
- removed the C40 at (59.8, 71.5)
- removed FID1, FID2, FID3: Fiducial_1mm_Mask2mm, Fiducial_1mm_Mask2mm
- added C40: 0.1u, Capacitor_SMD:C_0603_1608Metric_Pad1.08x0.95mm_HandSolder, F.Cu at (210.0, 105.4)
- added C40: 0.1u, Capacitor_SMD:C_0603_1608Metric_Pad1.08x0.95mm_HandSolder, F.Cu at (42.6, 56.8)
- L1: footprint ProtoFlow.pretty:Yageo_Pulse_PA4342_10.3x11.5mm -> PA4342.682NLT:Yageo_Pulse_PA4342_10.3x11.5mm
- moved D11 145.6 mm to (205.3, 105.4), turned to -90 degrees
- moved TP8 142.9 mm to (164.3, 78.9)
- moved TP7 141.3 mm to (161.2, 85.9)
- moved TP6 140.7 mm to (161.1, 78.8)
- moved Q7 140.3 mm to (216.4, 110.0), turned to 180 degrees
- moved D10 139.6 mm to (198.9, 105.4)
- moved C39 138.9 mm to (195.3, 103.7)
- moved C41 138.2 mm to (219.6, 105.9), turned to 0 degrees
- moved Q6 136.6 mm to (211.6, 110.0), turned to 180 degrees
- moved R24 136.5 mm to (220.5, 108.5), turned to -90 degrees
- moved C25 135.0 mm to (192.1, 82.5)
- moved C31 132.7 mm to (201.4, 86.1), turned to 90 degrees
- moved C26 131.8 mm to (192.1, 85.0)
- moved C28 131.7 mm to (161.7, 70.2), turned to 90 degrees
- moved C32 131.5 mm to (203.9, 86.1), turned to 90 degrees
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Routing:
- net GND: track 297.7 -> 74.6 mm, vias 25 -> 0
- net VDDD: track 218.9 -> 32.0 mm, vias 7 -> 0
- net /IOUT_CSN_0: track 116.2 -> 7.70 mm, vias 4 -> 0
- net /IOUT_CSP_0: track 96.2 -> 29.4 mm, vias 8 -> 0
- net /Vin: track 64.7 -> 0.00 mm, vias 3 -> 0
- net PVIN_0: track 89.5 -> 26.2 mm, vias 2 -> 0
- net /SW2_1: track 85.7 -> 22.6 mm, vias 3 -> 0
- net Net-(C44-Pad2): track 62.3 -> 1.82 mm, vias 2 -> 0
- net Net-(J3-Pin_1): track 55.3 -> 0.00 mm, vias 1 -> 0
- net Net-(C9-Pad1): track 84.1 -> 29.8 mm, vias 2 -> 0
- net /COIL_SNS: track 33.8 -> 87.6 mm
- net /LG1_0: track 52.6 -> 3.16 mm
- net /HPI_I2C_SCL: track 52.3 -> 90.4 mm, vias 1 -> 0
- net /ASK_OUT: track 59.2 -> 23.1 mm, vias 2 -> 0
- net /ASK_I_N: track 34.5 -> 0.00 mm
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- removed copper zone on F.Cu, net /IIN_CSN_0
- removed copper zone on F.Cu, net /SW1_0
- removed copper zone on F.Cu, net PVIN_0
Other:
- board outline removed
